File: heizungsregler.sch (KiCad schematic (older format))
At the start: 22 parts, among them J101 RPi_GPIO, J102 Conn_01x03_Male, J103 Conn_01x02, J104 Conn_01x03_Male, J105 Conn_01x04_Male, U101 oled_0.96\", U102 DS18B20

Commit message: Änderungen nach Review, Layout fertig
Connections:
- net ENC_#RESET: now reaches J101.11 (GPIO17)
Changed lines of the file:
@@
 F5 "ENC_#CS" I L 3300 5450 50
 F6 "ENC_#INT" O L 3300 5650 50
+F7 "ENC_#RESET" I L 3300 5550 50
 $EndSheet
 Wire Wire Line
@@
 Wire Wire Line
 	8050 1350 8700 1350
+Text Label 2850 5550 0    50   ~ 0
+ENC_#RESET
+Wire Wire Line
+	3300 5550 2850 5550
+Text Label 1750 2050 0    50   ~ 0
+ENC_#RESET
+Wire Wire Line
+	1750 2050 2500 2050
 $EndSCHEMATC

Commit message: Bauteilwerte beim Bestücken angepasst
Parts:
- C101: value C -> 100N
- R101: value R -> 4K7
- R104: value R -> 0R0
Changed lines of the file:
@@
 P 7250 4200
 F 0 "R101" H 7320 4246 50  0000 L CNN
-F 1 "R" H 7320 4155 50  0000 L CNN
+F 1 "4K7" H 7320 4155 50  0000 L CNN
 F 2 "Resistor_SMD:R_0603_1608Metric" V 7180 4200 50  0001 C CNN
 F 3 "~" H 7250 4200 50  0001 C CNN
@@
 P 5900 5150
 F 0 "C101" H 6015 5196 50  0000 L CNN
-F 1 "C" H 6015 5105 50  0000 L CNN
+F 1 "100N" H 6015 5105 50  0000 L CNN
 F 2 "Capacitor_SMD:C_0603_1608Metric" H 5938 5000 50  0001 C CNN
 F 3 "~" H 5900 5150 50  0001 C CNN
@@
 P 6750 4200
 F 0 "R104" H 6820 4246 50  0000 L CNN
-F 1 "R" H 6820 4155 50  0000 L CNN
+F 1 "0R0" H 6820 4155 50  0000 L CNN
 F 2 "Resistor_SMD:R_0603_1608Metric" V 6680 4200 50  0001 C CNN
 F 3 "~" H 6750 4200 50  0001 C CNN
