File: mbus.sch (KiCad schematic (older format))
At the start: 28 parts, among them J301 Conn_01x02_Male, Q301 BC847, Q302 BC847, Q303 BCP51, U301 MC34063AD

Commit message: Schaltplan weitergemacht, Footprints zugeordnet
Parts:
- C301, C303, C304: footprint (none) -> Capacitor_SMD:C_1210_3225Metric
- C302: footprint (none) -> Capacitor_SMD:C_0603_1608Metric
- D301: footprint (none) -> Diode_SMD:D_SOD-123
- F301: footprint (none) -> Fuse:Fuse_1812_4532Metric
- J301: footprint (none) -> Connector_PinHeader_2.54mm:PinHeader_1x02_P2.54mm_Vertical
- L301: footprint (none) -> Inductor_SMD:L_Bourns-SRN4018
- L302: value 150U -> 1U; footprint (none) -> Inductor_SMD:L_1206_3216Metric
- R301, R302, R303, R304, R305, R306, R307, R308, R309, R310, R311, R312, R313, R314, R315: footprint (none) -> Resistor_SMD:R_0603_1608Metric
Changed lines of the file:
@@
 F 0 "J301" H 6673 1730 50  0000 R CNN
 F 1 "Conn_01x02_Male" H 6673 1821 50  0000 R CNN
-F 2 "" H 6700 1850 50  0001 C CNN
+F 2 "Connector_PinHeader_2.54mm:PinHeader_1x02_P2.54mm_Vertical" H 6700 1850 50  0001 C CNN
 F 3 "~" H 6700 1850 50  0001 C CNN
 	1    6700 1850
@@
 F 0 "R313" V 4543 6200 50  0000 C CNN
 F 1 "22K" V 4634 6200 50  0000 C CNN
-F 2 "" V 4680 6200 50  0001 C CNN
+F 2 "Resistor_SMD:R_0603_1608Metric" V 4680 6200 50  0001 C CNN
 F 3 "~" H 4750 6200 50  0001 C CNN
 	1    4750 6200
@@
 F 0 "C301" H 1965 5996 50  0000 L CNN
 F 1 "22U" H 1965 5905 50  0000 L CNN
-F 2 "" H 1888 5800 50  0001 C CNN
+F 2 "Capacitor_SMD:C_1210_3225Metric" H 1888 5800 50  0001 C CNN
 F 3 "~" H 1850 5950 50  0001 C CNN
 	1    1850 5950
@@
 F 0 "D301" H 4600 5684 50  0000 C CNN
 F 1 "D_Schottky" H 4600 5775 50  0000 C CNN
-F 2 "" H 4600 5900 50  0001 C CNN
+F 2 "Diode_SMD:D_SOD-123" H 4600 5900 50  0001 C CNN
 F 3 "~" H 4600 5900 50  0001 C CNN
 	1    4600 5900
@@
 F 0 "L301" H 4203 5696 50  0000 L CNN
 F 1 "150U" H 4203 5605 50  0000 L CNN
-F 2 "" H 4150 5650 50  0001 C CNN
+F 2 "Inductor_SMD:L_Bourns-SRN4018" H 4150 5650 50  0001 C CNN
 F 3 "~" H 4150 5650 50  0001 C CNN
 	1    4150 5650
@@
 F 0 "C302" H 2315 6346 50  0000 L CNN
 F 1 "330P" H 2315 6255 50  0000 L CNN
-F 2 "" H 2238 6150 50  0001 C CNN
+F 2 "Capacitor_SMD:C_0603_1608Metric" H 2238 6150 50  0001 C CNN
 F 3 "~" H 2200 6300 50  0001 C CNN
 	1    2200 6300
@@
 F 0 "C303" H 5365 6496 50  0000 L CNN
 F 1 "47U" H 5365 6405 50  0000 L CNN
-F 2 "" H 5288 6300 50  0001 C CNN
+F 2 "Capacitor_SMD:C_1210_3225Metric" H 5288 6300 50  0001 C CNN
 F 3 "~" H 5250 6450 50  0001 C CNN
 	1    5250 6450
@@
 F 0 "R301" V 1143 5300 50  0000 C CNN
 F 1 "0R00" V 1234 5300 50  0000 C CNN
-F 2 "" V 1280 5300 50  0001 C CNN
+F 2 "Resistor_SMD:R_0603_1608Metric" V 1280 5300 50  0001 C CNN
 F 3 "~" H 1350 5300 50  0001 C CNN
 	1    1350 5300
@@
 F 0 "R302" V 1143 5700 50  0000 C CNN
 F 1 "0R00" V 1234 5700 50  0000 C CNN
-F 2 "" V 1280 5700 50  0001 C CNN
+F 2 "Resistor_SMD:R_0603_1608Metric" V 1280 5700 50  0001 C CNN
 F 3 "~" H 1350 5700 50  0001 C CNN
 	1    1350 5700
@@
 F 0 "R305" V 2693 5250 50  0000 C CNN
 F 1 "0R47" V 2784 5250 50  0000 C CNN
-F 2 "" V 2830 5250 50  0001 C CNN
+F 2 "Resistor_SMD:R_0603_1608Metric" V 2830 5250 50  0001 C CNN
 F 3 "~" H 2900 5250 50  0001 C CNN
 	1    2900 5250
@@
 F 0 "R306" V 3443 5800 50  0000 C CNN
 F 1 "180" V 3534 5800 50  0000 C CNN
-F 2 "" V 3580 5800 50  0001 C CNN
+F 2 "Resistor_SMD:R_0603_1608Metric" V 3580 5800 50  0001 C CNN
 F 3 "~" H 3650 5800 50  0001 C CNN
 	1    3650 5800
@@
 F 0 "R310" V 3993 6200 50  0000 C CNN
 F 1 "100K" V 4084 6200 50  0000 C CNN
-F 2 "" V 4130 6200 50  0001 C CNN
+F 2 "Resistor_SMD:R_0603_1608Metric" V 4130 6200 50  0001 C CNN
 F 3 "~" H 4200 6200 50  0001 C CNN
 	1    4200 6200
@@
 F 0 "R307" H 3680 6404 50  0000 R CNN
 F 1 "4k7" H 3680 6495 50  0000 R CNN
-F 2 "" V 3680 6450 50  0001 C CNN
+F 2 "Resistor_SMD:R_0603_1608Metric" V 3680 6450 50  0001 C CNN
 F 3 "~" H 3750 6450 50  0001 C CNN
 	1    3750 6450
@@
 F 0 "C304" H 6215 6496 50  0000 L CNN
 F 1 "47U" H 6215 6405 50  0000 L CNN
-F 2 "" H 6138 6300 50  0001 C CNN
+F 2 "Capacitor_SMD:C_1210_3225Metric" H 6138 6300 50  0001 C CNN
 F 3 "~" H 6100 6450 50  0001 C CNN
 	1    6100 6450
@@
 P 5650 6200
 F 0 "L302" V 5840 6200 50  0000 C CNN
-F 1 "150U" V 5749 6200 50  0000 C CNN
-F 2 "" H 5650 6200 50  0001 C CNN
+F 1 "1U" V 5749 6200 50  0000 C CNN
+F 2 "Inductor_SMD:L_1206_3216Metric" H 5650 6200 50  0001 C CNN
 F 3 "~" H 5650 6200 50  0001 C CNN
 	1    5650 6200
@@
 F 0 "F301" V 6403 6200 50  0000 C CNN
 F 1 "Fuse" V 6494 6200 50  0000 C CNN
-F 2 "" V 6530 6200 50  0001 C CNN
+F 2 "Fuse:Fuse_1812_4532Metric" V 6530 6200 50  0001 C CNN
 F 3 "~" H 6600 6200 50  0001 C CNN
 	1    6600 6200
@@
 F 0 "R303" V 1893 2400 50  0000 C CNN
 F 1 "1K" V 1984 2400 50  0000 C CNN
-F 2 "" V 2030 2400 50  0001 C CNN
+F 2 "Resistor_SMD:R_0603_1608Metric" V 2030 2400 50  0001 C CNN
 F 3 "~" H 2100 2400 50  0001 C CNN
 	1    2100 2400
@@
 F 0 "R304" V 1893 3150 50  0000 C CNN
 F 1 "1K" V 1984 3150 50  0000 C CNN
-F 2 "" V 2030 3150 50  0001 C CNN
+F 2 "Resistor_SMD:R_0603_1608Metric" V 2030 3150 50  0001 C CNN
 F 3 "~" H 2100 3150 50  0001 C CNN
 	1    2100 3150
@@
 F 0 "R309" H 3780 2504 50  0000 R CNN
 F 1 "22K" H 3780 2595 50  0000 R CNN
-F 2 "" V 3780 2550 50  0001 C CNN
+F 2 "Resistor_SMD:R_0603_1608Metric" V 3780 2550 50  0001 C CNN
 F 3 "~" H 3850 2550 50  0001 C CNN
 	1    3850 2550
@@
 F 0 "R308" H 3780 1604 50  0000 R CNN
 F 1 "39K" H 3780 1695 50  0000 R CNN
-F 2 "" V 3780 1650 50  0001 C CNN
+F 2 "Resistor_SMD:R_0603_1608Metric" V 3780 1650 50  0001 C CNN
 F 3 "~" H 3850 1650 50  0001 C CNN
 	1    3850 1650
@@
 F 0 "R314" H 5580 1604 50  0000 R CNN
 F 1 "220K" H 5580 1695 50  0000 R CNN
-F 2 "" V 5580 1650 50  0001 C CNN
+F 2 "Resistor_SMD:R_0603_1608Metric" V 5580 1650 50  0001 C CNN
 F 3 "~" H 5650 1650 50  0001 C CNN
 	1    5650 1650
@@
 F 0 "R315" H 5580 2504 50  0000 R CNN
 F 1 "82R" H 5580 2595 50  0000 R CNN
-F 2 "" V 5580 2550 50  0001 C CNN
+F 2 "Resistor_SMD:R_0603_1608Metric" V 5580 2550 50  0001 C CNN
 F 3 "~" H 5650 2550 50  0001 C CNN
 	1    5650 2550
@@
 F 0 "R312" H 4280 2504 50  0000 R CNN
 F 1 "3K3" H 4280 2595 50  0000 R CNN
-F 2 "" V 4280 2550 50  0001 C CNN
+F 2 "Resistor_SMD:R_0603_1608Metric" V 4280 2550 50  0001 C CNN
 F 3 "~" H 4350 2550 50  0001 C CNN
 	1    4350 2550
@@
 F 0 "R311" H 4280 1604 50  0000 R CNN
 F 1 "33K" H 4280 1695 50  0000 R CNN
-F 2 "" V 4280 1650 50  0001 C CNN
+F 2 "Resistor_SMD:R_0603_1608Metric" V 4280 1650 50  0001 C CNN
 F 3 "~" H 4350 1650 50  0001 C CNN
 	1    4350 1650

Commit message: ENC28J60 platziert und geroutet
Parts:
- F301: value Fuse -> Fuse 2A
Changed lines of the file:
@@
 P 6600 6200
 F 0 "F301" V 6403 6200 50  0000 C CNN
-F 1 "Fuse" V 6494 6200 50  0000 C CNN
+F 1 "Fuse 2A" V 6494 6200 50  0000 C CNN
 F 2 "Fuse:Fuse_1812_4532Metric" V 6530 6200 50  0001 C CNN
 F 3 "~" H 6600 6200 50  0001 C CNN

Commit message: Design weiter bearbeitet
Parts:
- removed C301: 22U, Capacitor_SMD:C_1210_3225Metric, symbol Device:C
- removed C303: 47U, Capacitor_SMD:C_1210_3225Metric, symbol Device:C
- added C301: 22U, Capacitor_SMD:CP_Elec_6.3x5.7, symbol Device:CP
- added C303: 47U, Capacitor_SMD:CP_Elec_6.3x7.7, symbol Device:CP
- C304: value 47U -> 1U; footprint Capacitor_SMD:C_1210_3225Metric -> Capacitor_SMD:C_1206_3216Metric
Connections:
- net GND: now also C301.2, C303.2
- net at R301.1, R302.1, R305.2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: now also C301.1
- net at L302.1, R313.1: now also C303.1
Changed lines of the file:
@@
-$EndComp
-$Comp
-L Device:C C301
-U 1 1 5C09E68A
-P 1850 5950
-F 0 "C301" H 1965 5996 50  0000 L CNN
-F 1 "22U" H 1965 5905 50  0000 L CNN
-F 2 "Capacitor_SMD:C_1210_3225Metric" H 1888 5800 50  0001 C CNN
-F 3 "~" H 1850 5950 50  0001 C CNN
-	1    1850 5950
-	1    0    0    -1
 $EndComp
 $Comp
@@
 $EndComp
 $Comp
-L Device:C C303
-U 1 1 5C09EFB1
-P 5250 6450
-F 0 "C303" H 5365 6496 50  0000 L CNN
-F 1 "47U" H 5365 6405 50  0000 L CNN
-F 2 "Capacitor_SMD:C_1210_3225Metric" H 5288 6300 50  0001 C CNN
-F 3 "~" H 5250 6450 50  0001 C CNN
-	1    5250 6450
-	1    0    0    -1
-$EndComp
-$Comp
 L power:GND #PWR0303
 U 1 1 5C09F015
@@
 P 6100 6450
 F 0 "C304" H 6215 6496 50  0000 L CNN
-F 1 "47U" H 6215 6405 50  0000 L CNN
-F 2 "Capacitor_SMD:C_1210_3225Metric" H 6138 6300 50  0001 C CNN
+F 1 "1U" H 6215 6405 50  0000 L CNN
+F 2 "Capacitor_SMD:C_1206_3216Metric" H 6138 6300 50  0001 C CNN
 F 3 "~" H 6100 6450 50  0001 C CNN
 	1    6100 6450
@@
 Wire Wire Line
 	5350 2350 5650 2350
+$Comp
+L Device:CP C303
+U 1 1 5C1005E1
+P 5250 6450
+F 0 "C303" H 5368 6496 50  0000 L CNN
+F 1 "47U" H 5368 6405 50  0000 L CNN
+F 2 "Capacitor_SMD:CP_Elec_6.3x7.7" H 5288 6300 50  0001 C CNN
+F 3 "~" H 5250 6450 50  0001 C CNN
+	1    5250 6450
+	1    0    0    -1
+$EndComp
+$Comp
+L Device:CP C301
+U 1 1 5C105276
+P 1850 5950
+F 0 "C301" H 1968 5996 50  0000 L CNN
+F 1 "22U" H 1968 5905 50  0000 L CNN
+F 2 "Capacitor_SMD:CP_Elec_6.3x5.7" H 1888 5800 50  0001 C CNN
+F 3 "~" H 1850 5950 50  0001 C CNN
+	1    1850 5950
+	1    0    0    -1
+$EndComp
 $EndSCHEMATC

Commit message: Transistoren für Relais eingefügt, Pull-Ups für I2C, zusätzlicher Spannungseingang, Layout fertig
Connections:
- net at C303.1, L302.1, R313.1: now also D301.1 (K)
Changed lines of the file:
@@
 $Descr A4 11693 8268
 encoding utf-8
-Sheet 3 3
+Sheet 3 4
 Title ""
 Date ""
@@
 Connection ~ 3750 6200
 Wire Wire Line
-	4800 5900 5250 5900
-Wire Wire Line
 	5250 5900 5250 6200
 Wire Wire Line
@@
 	1    0    0    -1
 $EndComp
+Wire Wire Line
+	4750 5900 5250 5900
 $EndSCHEMATC

Commit message: Änderungen nach Review, Layout fertig
Parts:
- C302: value 330P -> 140P
- L301: value 150U -> 270U
- R305: value 0R47 -> 1R00
- R313: value 22K -> 26K9
Changed lines of the file:
@@
 P 4750 6200
 F 0 "R313" V 4543 6200 50  0000 C CNN
-F 1 "22K" V 4634 6200 50  0000 C CNN
+F 1 "26K9" V 4634 6200 50  0000 C CNN
 F 2 "Resistor_SMD:R_0603_1608Metric" V 4680 6200 50  0001 C CNN
 F 3 "~" H 4750 6200 50  0001 C CNN
@@
 P 4150 5650
 F 0 "L301" H 4203 5696 50  0000 L CNN
-F 1 "150U" H 4203 5605 50  0000 L CNN
+F 1 "270U" H 4203 5605 50  0000 L CNN
 F 2 "Inductor_SMD:L_Bourns-SRN4018" H 4150 5650 50  0001 C CNN
 F 3 "~" H 4150 5650 50  0001 C CNN
@@
 P 2200 6300
 F 0 "C302" H 2315 6346 50  0000 L CNN
-F 1 "330P" H 2315 6255 50  0000 L CNN
+F 1 "140P" H 2315 6255 50  0000 L CNN
 F 2 "Capacitor_SMD:C_0603_1608Metric" H 2238 6150 50  0001 C CNN
 F 3 "~" H 2200 6300 50  0001 C CNN
@@
 P 2900 5250
 F 0 "R305" V 2693 5250 50  0000 C CNN
-F 1 "0R47" V 2784 5250 50  0000 C CNN
+F 1 "1R00" V 2784 5250 50  0000 C CNN
 F 2 "Resistor_SMD:R_0603_1608Metric" V 2830 5250 50  0001 C CNN
 F 3 "~" H 2900 5250 50  0001 C CNN

Commit message: Bauteilwerte beim Bestücken angepasst
Parts:
- C302: value 140P -> 150P
- R313: value 26K9 -> 27k0
Changed lines of the file:
@@
 P 4750 6200
 F 0 "R313" V 4543 6200 50  0000 C CNN
-F 1 "26K9" V 4634 6200 50  0000 C CNN
+F 1 "27k0" V 4634 6200 50  0000 C CNN
 F 2 "Resistor_SMD:R_0603_1608Metric" V 4680 6200 50  0001 C CNN
 F 3 "~" H 4750 6200 50  0001 C CNN
@@
 P 2200 6300
 F 0 "C302" H 2315 6346 50  0000 L CNN
-F 1 "140P" H 2315 6255 50  0000 L CNN
+F 1 "150P" H 2315 6255 50  0000 L CNN
 F 2 "Capacitor_SMD:C_0603_1608Metric" H 2238 6150 50  0001 C CNN
 F 3 "~" H 2200 6300 50  0001 C CNN
